File: Illuminoti-board/A_Team_ECE411.kicad_pcb (KiCad board)
At the start: 2 copper layers, 16 parts, among them IC1 TPS61023_Boost_Converter, U1 LIS3DH_Accelerator, U2 RF522_RFID

Commit message: Add files via upload
Most recent schematic and pcb files. The footprint for the accelerometer is the most urgent thing to be adjusted and then general cleanup could be helpful if time allows.
Parts:
- removed C4: 100u, Capacitor_THT:CP_Radial_D6.3mm_P2.50mm
- removed L1: 1u, Inductor_THT:L_Axial_L11.0mm_D4.5mm_P5.08mm_Vertical_Fastron_MECC
- removed R1: 10k, Resistor_THT:R_Axial_DIN0207_L6.3mm_D2.5mm_P10.16mm_Horizontal
- removed R2: 723k, Resistor_THT:R_Axial_DIN0207_L6.3mm_D2.5mm_P10.16mm_Horizontal
- removed R3: 100k, Resistor_THT:R_Axial_DIN0207_L6.3mm_D2.5mm_P10.16mm_Horizontal
- removed R4: 330, Resistor_THT:R_Axial_DIN0207_L6.3mm_D2.5mm_P10.16mm_Horizontal
- removed U1: LIS3DH_Accelerator, Package_LGA:LGA-16_3x3mm_P0.5mm_LayoutBorder3x5y
- added D4: WS2812B-2020-LED, Connector_PinHeader_2.54mm:PinHeader_1x03_P2.54mm_Vertical, F.Cu at (181.5, 110.5)
- added FID4: FIDUCIAL_1MM, Adafruit LIS3DH:FIDUCIAL_1MM, F.Cu at (179.7, 52.1)
- added JP2: , Adafruit LIS3DH:1X06_ROUND_70, F.Cu at (177.9, 59.4)
- added JP3: , Adafruit LIS3DH:1X06_ROUND_70, F.Cu at (190.6, 59.4)
- added SW1: SW_Wuerth_450301014042, Connector_PinHeader_2.54mm:PinHeader_1x03_P2.54mm_Vertical, F.Cu at (213.0, 109.0)
- added U$1: MOUNTINGHOLE2.5, Adafruit LIS3DH:MOUNTINGHOLE_2.5_PLATED, F.Cu at (177.9, 69.6)
- added U$12: , Adafruit LIS3DH:ADAFRUIT_2.5MM, F.Cu at (189.1, 57.1)
- added U$17: MOUNTINGHOLE2.5, Adafruit LIS3DH:MOUNTINGHOLE_2.5_PLATED, F.Cu at (177.9, 49.3)
- added U$19: MOUNTINGHOLE2.5, Adafruit LIS3DH:MOUNTINGHOLE_2.5_PLATED, F.Cu at (190.6, 69.6)
- added U$21: MOUNTINGHOLE2.5, Adafruit LIS3DH:MOUNTINGHOLE_2.5_PLATED, F.Cu at (190.6, 49.3)
- D1: footprint LED_SMD:LED_WS2812B-2020_PLCC4_2.0x2.0mm -> Connector_PinHeader_2.54mm:PinHeader_1x03_P2.54mm_Vertical
- IC1: footprint Adafruit TPS61023:SOT563 -> Connector_PinHeader_2.54mm:PinHeader_1x04_P2.54mm_Vertical
- moved C1 93.0 mm to (153.0, 92.5)
- moved U2 87.9 mm to (253.5, 66.5), turned to 90 degrees
- moved C3 75.5 mm to (163.5, 114.0)
- moved C2 69.9 mm to (163.5, 120.5)
- moved IC1 49.6 mm to (205.5, 113.7)
- moved TP1 49.2 mm to (170.5, 107.5)
- moved TP2 49.2 mm to (170.5, 110.5)
- moved D1 45.9 mm to (176.5, 110.5)
- moved A1 43.4 mm to (166.0, 102.5), turned to 90 degrees
Connections:
- net /IO10 renamed /CS
- A1 pad 23: /IO11 -> unconnected-(A1-IO11-Pad23)
- A1 pad 3: unconnected-(A1-3V3-Pad3) -> Net-(SW1-B)
- A1 pad 6: unconnected-(A1-A1-Pad6) -> /IO11
- A1 pad 7: unconnected-(A1-A2-Pad7) -> Net-(A1-A2)
- D1 pad 3: Net-(D1-DIN) -> /IO11
- IC1 pad 1: Net-(IC1-FB) -> unconnected-(IC1-FB-Pad1)
- IC1 pad 2: Net-(IC1-EN) -> /IO6
- TP1 pad 1: Net-(U1-INT2) -> /INT2
Routing:
- net +BATT: track 0.00 -> 114.2 mm
- net GND: track 0.00 -> 102.3 mm, vias 0 -> 16
- net /IO6: track 0.00 -> 90.3 mm
- net /REST: track 0.00 -> 74.8 mm
- net +3.3V: track 0.00 -> 71.7 mm
- net /SCK: track 0.00 -> 63.4 mm
- net /MOSI: track 0.00 -> 57.8 mm
- net /MISO: track 0.00 -> 51.9 mm
- net /CS: track 0.00 -> 46.2 mm
- net Net-(SW1-B): track 0.00 -> 44.6 mm
- net Net-(A1-A2): track 0.00 -> 16.0 mm
- net /IO11: track 0.00 -> 14.2 mm
- net /A0: track 0.00 -> 10.3 mm
- net +5V: track 0.00 -> 6.50 mm
- added copper zone on B.Cu, net (none)
- added copper zone on B.Cu, net GND
- added copper zone on F.Cu, net GND
Other:
- board outline added: 93 x 82.5 mm
- board text added: "3-axis Accelerometer ±2g/±4g/±8g I2C addr 0x18"
- board text added: "LIS3DH"
- board text added: "VLogic/Vcc: 3-5VDC"
- board text added: "addr"

Commit message: Add files via upload
edited footprints, resolved DRC errors
Parts:
- removed FID4: FIDUCIAL_1MM, Adafruit LIS3DH:FIDUCIAL_1MM
- removed U$1, U$17, U$19, U$21: MOUNTINGHOLE2.5, Adafruit LIS3DH:MOUNTINGHOLE_2.5_PLATED
- removed U$12: , Adafruit LIS3DH:ADAFRUIT_2.5MM
- added SW2: SW_Wuerth_450301014042, Connector_PinHeader_2.54mm:PinHeader_1x03_P2.54mm_Vertical, F.Cu at (173.5, 74.0)
- JP2, JP3: value (none) -> HEADER-1X670MIL; footprint Adafruit LIS3DH:1X06_ROUND_70 -> Connector_PinHeader_2.54mm:PinHeader_1x06_P2.54mm_Vertical
- U2: footprint CEG006900:MODULE_CEG006900 -> Connector_PinHeader_2.54mm:PinHeader_1x08_P2.54mm_Vertical
- moved U2 48.0 mm to (221.7, 102.5), turned to 180 degrees
- moved TP1 43.5 mm to (149.6, 69.3), turned to 90 degrees
- moved JP2 41.6 mm to (144.8, 84.7), turned to 180 degrees
- moved JP3 35.4 mm to (157.5, 72.0), turned to 0 degrees
- moved C1 23.9 mm to (153.7, 116.4)
- moved C2 22.9 mm to (186.4, 121.2)
- moved D4 18.4 mm to (163.5, 114.5), turned to 90 degrees
- moved D1 13.3 mm to (163.2, 109.7), turned to 90 degrees
- moved C3 12.0 mm to (173.4, 120.8)
- moved TP2 9.55 mm to (179.6, 107.6)
- moved SW1 5.26 mm to (214.5, 114.0)
Connections:
- net ADC1 renamed /ADC1
- net ADC2 renamed /ADC2
- net ADC3 renamed /ADC3
- A1 pad 21: /IO9 -> /CS
- A1 pad 22: /CS -> /IO10
- A1 pad 27: unconnected-(A1-EN-Pad27) -> Net-(A1-EN)
- A1 pad 28: +BATT -> unconnected-(A1-VBAT-Pad28)
- A1 pad 3: Net-(SW1-B) -> Net-(A1-3V3-Pad3)
- C1 pad 1: +BATT -> +3.3V
- D1 pad 1: unconnected-(D1-DOUT-Pad1) -> +5V
- D1 pad 2: GND -> /IO11
- D1 pad 3: /IO11 -> GND
- D4 pad 1: unconnected-(D4-DOUT-Pad1) -> +5V
- D4 pad 2: GND -> Net-(A1-A2)
- D4 pad 3: Net-(A1-A2) -> GND
- IC1 pad 1: unconnected-(IC1-FB-Pad1) -> +3.3V
- IC1 pad 2: /IO6 -> GND
- IC1 pad 3: +BATT -> +5V
- IC1 pad 4: GND -> /IO6
- JP2 pad 1: CS -> /CS
- JP2 pad 2: SDO -> /MISO
- JP2 pad 6: INT2 -> /INT2
- JP3 pad 1: VCC -> Net-(A1-3V3-Pad3)
- JP3 pad 2: 3.3V -> unconnected-(JP3-Pad2)
- JP3 pad 4: SCL -> /SCK
- JP3 pad 5: SDA -> /MOSI
- JP3 pad 6: INT1 -> /A0
- SW1 pad 1: Net-(SW1-B) -> GND
- SW1 pad 3: GND -> +3.3V
- U2 pad 8: /CS -> /IO10
Routing:
- net +BATT: track 114.2 -> 0.00 mm
- net GND: track 102.3 -> 0.04 mm, vias 16 -> 17
- net +3.3V: track 71.7 -> 128.5 mm
- net Net-(A1-3V3-Pad3): track 0.00 -> 51.8 mm
- net +5V: track 6.50 -> 52.5 mm
- net /MISO: track 51.9 -> 97.5 mm
- net Net-(SW1-B): track 44.6 -> 0.00 mm
- net /IO10: track 0.00 -> 33.2 mm
- net /A0: track 10.3 -> 38.7 mm
- net /MOSI: track 57.8 -> 81.3 mm
- net /CS: track 46.2 -> 64.0 mm
- net /SCK: track 63.4 -> 80.4 mm
- net Net-(A1-EN): track 0.00 -> 10.3 mm
- net /REST: track 74.8 -> 68.1 mm
- net /IO6: track 90.3 -> 96.7 mm
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- removed copper zone on B.Cu, net (none)
Other:
- board size 93 x 82.5 mm -> 87.9 x 59.2 mm
- board text added: "10"
- board text added: "11"
- board text added: "12"
- board text added: "13"
- board text added: "3 1 2"
- board text added: "3 GND 1 EN 2 3V"
- board text added: "3V Vin"
- board text added: "5V Vin"
- board text added: "5V Vout"
- board text added: "9 6 5 SCL SDA"
- board text added: "A2 A3 A4 A5 SCK MOSI MISO RX TX DB"
- board text added: "BATT"
- board text added: "CS"
- board text added: "Din"
- board text added: "EN"
- board text added: "GND"
- board text added: "I2 A3 A2 A1 SD0 CS"
- board text added: "MISO"
- board text added: "MOSI"
- board text added: "PWR"
- board text added: "REST"
- board text added: "REST 3V 3V GND A0 A1"
- board text added: "SCK"
- board text added: "Team 1 V1 Nov. 20, 2025"
- board text added: "USB"
- board text added: "Vin/3V 3V/X GND/GND SCK/SCK SDA/MOSI IN/A0"
- board text added: "X"
- board text removed: "3-axis Accelerometer ±2g/±4g/±8g I2C addr 0x18"
- board text removed: "LIS3DH"
- board text removed: "VLogic/Vcc: 3-5VDC"
- board text removed: "addr"
