File: Illuminoti-board/A_Team_ECE411.kicad_sch (KiCad schematic)
At the start: 16 parts, among them IC1 TPS61023_Boost_Converter, U1 LIS3DH_Accelerator, U2 RF522_RFID

Commit message: Add files via upload
Most recent schematic and pcb files. The footprint for the accelerometer is the most urgent thing to be adjusted and then general cleanup could be helpful if time allows.
Parts:
- removed C4: 100u, Capacitor_THT:CP_Radial_D6.3mm_P2.50mm, symbol Device:C_Small
- removed L1: 1u, Inductor_THT:L_Axial_L11.0mm_D4.5mm_P5.08mm_Vertical_Fastron_MECC, symbol Device:L
- removed R1: 10k, Resistor_THT:R_Axial_DIN0207_L6.3mm_D2.5mm_P10.16mm_Horizontal, symbol Device:R_US
- removed R2: 723k, Resistor_THT:R_Axial_DIN0207_L6.3mm_D2.5mm_P10.16mm_Horizontal, symbol Device:R_US
- removed R3: 100k, Resistor_THT:R_Axial_DIN0207_L6.3mm_D2.5mm_P10.16mm_Horizontal, symbol Device:R_US
- removed R4: 330, Resistor_THT:R_Axial_DIN0207_L6.3mm_D2.5mm_P10.16mm_Horizontal, symbol Device:R_US
- removed U1: LIS3DH_Accelerator, Package_LGA:LGA-16_3x3mm_P0.5mm_LayoutBorder3x5y, symbol Sensor_Motion:LIS3DH
- added C5, C6: 10uF, Capacitor_SMD:C_1206_3216Metric_Pad1.33x1.80mm_HandSolder, symbol Adafruit LIS3DH-eagle-import:CAP_CERAMIC0805-NOOUTLINE
- added C7: 0.1uF, Capacitor_SMD:C_1206_3216Metric_Pad1.33x1.80mm_HandSolder, symbol Adafruit LIS3DH-eagle-import:CAP_CERAMIC0603_NO
- added CONN3, CONN4: STEMMA_I2C_QT, Adafruit LIS3DH:JST_SH4, symbol Adafruit LIS3DH-eagle-import:STEMMA_I2C_QT
- added D2: 1N4148, PCM_LED_THT_AKL:LED_D5.0mm_Horizontal_O6.35mm_Z15.0mm, symbol Adafruit LIS3DH-eagle-import:DIODESOD-323
- added D3: GREEN, PCM_LED_THT_AKL:LED_D5.0mm_Horizontal_O6.35mm_Z15.0mm, symbol Adafruit LIS3DH-eagle-import:LED0603_NOOUTLINE
- added D4: WS2812B-2020-LED, Connector_PinHeader_2.54mm:PinHeader_1x03_P2.54mm_Vertical, symbol LED:WS2812B-2020
- added JP2, JP3: HEADER-1X670MIL, Adafruit LIS3DH:1X06_ROUND_70, symbol Adafruit LIS3DH-eagle-import:HEADER-1X670MIL
- added Q2: BSS138, Adafruit LIS3DH:SOT363, symbol Adafruit LIS3DH-eagle-import:MOSFET-N_DUAL
- added R5, R6: 10K, Resistor_THT:R_Axial_DIN0207_L6.3mm_D2.5mm_P10.16mm_Horizontal, symbol Adafruit LIS3DH-eagle-import:RESISTOR_4PACK
- added SJ1: SOLDERJUMPER, Adafruit LIS3DH:SOLDERJUMPER_ARROW_NOPASTE, symbol Adafruit LIS3DH-eagle-import:SOLDERJUMPER
- added SW1: SW_Wuerth_450301014042, Connector_PinHeader_2.54mm:PinHeader_1x03_P2.54mm_Vertical, symbol Switch:SW_Wuerth_450301014042
- added U3: AP2112K-3.3, PCM_Package_TO_SOT_SMD_AKL:Diodes_SOT-89-5, symbol Adafruit LIS3DH-eagle-import:VREG_SOT23-5
- added U4: LIS3DHTR, Package_LGA:LGA-16_3x3mm_P0.5mm_LayoutBorder3x5y, symbol Adafruit LIS3DH-eagle-import:ACCEL_LIS3DHTR
- D1: footprint LED_SMD:LED_WS2812B-2020_PLCC4_2.0x2.0mm -> Connector_PinHeader_2.54mm:PinHeader_1x03_P2.54mm_Vertical
- IC1: footprint Adafruit TPS61023:SOT563 -> Connector_PinHeader_2.54mm:PinHeader_1x04_P2.54mm_Vertical
Connections:
- net +5V: now also D4.4 (VDD)
- net GND: now also C5.2, C6.2, C7.2, CONN3.1 (GND), CONN4.1 (GND), D3.C, D4.2 (VSS), JP3.3, R5.6 (2), SW1.3 (A), U3.2 (GND), U4.10 (RES(GND)), U4.12 (GND@2), U4.5 (GND@1)
- net IO11: now also A1.6 (A1), D1.3 (DIN); no longer A1.23 (IO11)
- net IO6: now also IC1.2 (EN), SW1.2 (C)
- net MISO: now also JP2.2, R5.3 (1), SJ1.2, U4.7 (SDO)
- net MOSI: now also CONN3.3 (SDA), CONN4.3 (SDA), JP3.5, Q2.3 (D), R6.6 (2)
- net SCK: now also CONN3.4 (SCL), CONN4.4 (SCL), JP3.4, Q2.6 (D), R6.8 (2)
- net at A1.3 (3V3): now also SW1.1 (B)
- net at A1.7 (A2): now also D4.3 (DIN)
- net INT2: now reaches TP1.1
- net INT2: now also JP2.6, U4.9 (INT2)
- net A0 renamed RFID_INT1
- net RFID_INT1: now also JP3.6, U4.11 (INT1)
- net IO10 renamed CS
- net CS: now also D2.C, JP2.1
- new net: D2.A, R5.2 (1), U4.8 (CS)
- new net: D3.A, R5.4 (1)
- new net 3.3V: C6.1, C7.1, JP3.2, Q2.2 (G), Q2.5 (G), R5.1, R5.5 (2), R5.7 (2), R5.8 (2), R6.2 (1), R6.4 (1), SJ1.1, U3.5 (OUT), U4.1 (VDDIO), U4.14 (VDD)
- new net ADC1: JP2.3, U4.16 (ADC1)
- new net ADC2: JP2.4, U4.15 (ADC2)
- new net ADC3: JP2.5, U4.13 (ADC3)
- new net SCL_3V: Q2.1 (S), R6.7 (2), U4.4 (SCL)
- new net SDA_3V: Q2.4 (S), R6.5 (2), U4.6 (SDA)
- new net VCC: C5.1, CONN3.2 (V+), CONN4.2 (V+), JP3.1, R6.1, R6.3 (1), U3.1 (IN), U3.3 (EN)
Other:
- note added: "* CS needs to be set off board to select SPI or I2C"
- note added: "Bus Selection"
- note added: "CS High = I2C, Low = SPI"
- note added: "D"
- note added: "Defaults to I2C as-is (R8)"
- note added: "G"
- note added: "I2C"
- note added: "I2C Pullups & Shift"
- note added: "ON LED"
- note added: "Power supply"
- note added: "S"
- note added: "SCL (Pin 4) = Serial Clock"
- note added: "SD0 (Pin 7) = SA0/Address LSB"
- note added: "SDA (Pin 6) = Data In (MOSI)"
- note added: "SDA (Pin 6) = Serial Data"
- note added: "SDO (Pin 7) = Data Out (MISO)"
- note added: "SDO pulled low by default (R1) to set I2C address LSB to 0"
- note added: "SPI"
- note added: "STEMMA/I2C Headers"
- note added: "Set SJ1 to make I2C"
- note added: "address LSB 1"
- moved on the sheet: A1, C1, C2, C3, D1, IC1, TP1, TP2, U2

Commit message: Add files via upload
edited footprints, resolved DRC errors
Parts:
- removed C5, C6: 10uF, Capacitor_SMD:C_1206_3216Metric_Pad1.33x1.80mm_HandSolder, symbol Adafruit LIS3DH-eagle-import:CAP_CERAMIC0805-NOOUTLINE
- removed C7: 0.1uF, Capacitor_SMD:C_1206_3216Metric_Pad1.33x1.80mm_HandSolder, symbol Adafruit LIS3DH-eagle-import:CAP_CERAMIC0603_NO
- removed CONN3, CONN4: STEMMA_I2C_QT, Adafruit LIS3DH:JST_SH4, symbol Adafruit LIS3DH-eagle-import:STEMMA_I2C_QT
- removed D2: 1N4148, PCM_LED_THT_AKL:LED_D5.0mm_Horizontal_O6.35mm_Z15.0mm, symbol Adafruit LIS3DH-eagle-import:DIODESOD-323
- removed D3: GREEN, PCM_LED_THT_AKL:LED_D5.0mm_Horizontal_O6.35mm_Z15.0mm, symbol Adafruit LIS3DH-eagle-import:LED0603_NOOUTLINE
- removed Q2: BSS138, Adafruit LIS3DH:SOT363, symbol Adafruit LIS3DH-eagle-import:MOSFET-N_DUAL
- removed R5, R6: 10K, Resistor_THT:R_Axial_DIN0207_L6.3mm_D2.5mm_P10.16mm_Horizontal, symbol Adafruit LIS3DH-eagle-import:RESISTOR_4PACK
- removed SJ1: SOLDERJUMPER, Adafruit LIS3DH:SOLDERJUMPER_ARROW_NOPASTE, symbol Adafruit LIS3DH-eagle-import:SOLDERJUMPER
- removed U3: AP2112K-3.3, PCM_Package_TO_SOT_SMD_AKL:Diodes_SOT-89-5, symbol Adafruit LIS3DH-eagle-import:VREG_SOT23-5
- removed U4: LIS3DHTR, Package_LGA:LGA-16_3x3mm_P0.5mm_LayoutBorder3x5y, symbol Adafruit LIS3DH-eagle-import:ACCEL_LIS3DHTR
- added SW2: SW_Wuerth_450301014042, Connector_PinHeader_2.54mm:PinHeader_1x03_P2.54mm_Vertical, symbol Switch:SW_Wuerth_450301014042
- JP2, JP3: footprint Adafruit LIS3DH:1X06_ROUND_70 -> Connector_PinHeader_2.54mm:PinHeader_1x06_P2.54mm_Vertical
- U2: footprint CEG006900:MODULE_CEG006900 -> Connector_PinHeader_2.54mm:PinHeader_1x08_P2.54mm_Vertical
Connections:
- net IO9 is gone; now on net CS: A1.21 (IO9)
- net VCC is gone; now on an unnamed net: JP3.1
- net +3.3V: now also C1.1, IC1.1 (VIN), SW1.3 (3V)
- net +5V: now also D1.1 (VDD), D4.1 (VDD), IC1.3 (VOUT); no longer D1.4 (VDD), D4.4 (VDD), IC1.6 (VOUT)
- net CS: no longer A1.22 (IO10), U2.8 (SS/SDA/RX)
- net GND: now also D1.3 (GND), D4.3 (GND), IC1.2 (GND), SW1.1 (GND), SW2.2 (B); no longer D1.2 (VSS), D4.2 (VSS), IC1.4 (GND), SW1.3 (A)
- net IO11: now also D1.2 (DIN); no longer D1.3 (DIN)
- net IO6: now also IC1.4 (EN); no longer IC1.2 (EN)
- net at A1.27 (EN): now also SW2.1 (A)
- net at A1.3 (3V3): no longer SW1.1 (B)
- net at A1.7 (A2): now also D4.2 (DIN); no longer D4.3 (DIN)
- removed net +BATT: A1.28 (VBAT), C1.1, IC1.3 (VIN)
- net 3.3V: no longer names the net of JP3.2
- net RFID_INT1 renamed A0
- new net IO10: A1.22 (IO10), U2.8 (SS/SDA/RX)
- no-connect marks 21 -> 24
Other:
- note added: "I2/ TP1 A3 A2 A1 MISO/SDO CS / I09"
- note added: "Vin/ESP32 P3 3V NC GND SCL/SCK SDA/MOSI INT/A0"
- note added: "turn off LED's"
- note added: "turn off system"
- note removed: "* CS needs to be set off board to select SPI or I2C"
- note removed: "Bus Selection"
- note removed: "D"
- note removed: "G"
- note removed: "I2C Pullups & Shift"
- note removed: "ON LED"
- note removed: "Power supply"
- note removed: "S"
- note removed: "STEMMA/I2C Headers"
- note removed: "Set SJ1 to make I2C"
- note removed: "address LSB 1"
- moved on the sheet: A1, JP3, SW1, TP1, TP2
